Commit message: updated xacro files

File: urdfs/tracer_joints.xacro (robot description, xacro)
@@ -11,4 +11,9 @@
         <parent link="base_link"/>
         <child link="inertial_link"/>
+    </joint>
+    <joint name="rig_joint" type="fixed">
+        <origin xyz="0 0 0.015" rpy="0 0 0"/>
+        <parent link="base_link"/>
+        <child link="akula_rig_link"/>
     </joint>
     <!-- ************************************************** -->

File: urdfs/tracer_links.xacro (robot description, xacro)
@@ -41,4 +41,7 @@
         <mesh filename="file://$(find tracer_ign_sim)/models/tracer/meshes/tracer_wheel.dae"/>
     </xacro:macro>
+    <xacro:macro name="akula_rig">
+        <mesh filename="file://$(find tracer_ign_sim)/models/tracer/meshes/tracer_sensor_rig.stl" scale="0.001 0.001 0.001"/>
+    </xacro:macro>
     <!-- Initial Link -->
     <link name="inertial_link">
@@ -279,3 +282,23 @@
         </collision>
     </link>
+    <link name="akula_rig_link">
+        <visual>
+            <geometry>
+                <xacro:akula_rig></xacro:akula_rig>
+            </geometry>
+            <material name="rig">
+                <color rgba="0.1 0.1 0.1 1"/>
+            </material>
+        </visual>
+        <inertial>
+            <mass value="1" />
+            <origin xyz="0 0 0" />
+            <inertia ixx="0.3" ixy="0" ixz="0" iyy="0.3" iyz="0" izz="0.3" />
+        </inertial>
+        <collision>
+            <geometry>
+                <xacro:akula_rig></xacro:akula_rig>
+            </geometry>
+        </collision>
+    </link>
 </robot>

Commit message: fin is added to the top of Tracer

File: urdfs/tracer_joints.xacro (robot description, xacro)
@@ -12,8 +12,8 @@
         <child link="inertial_link"/>
     </joint>
-    <joint name="rig_joint" type="fixed">
-        <origin xyz="0 0 0.015" rpy="0 0 0"/>
+    <joint name="fin_joint" type="fixed">
+        <origin xyz="0 0 -0.15" rpy="0 0 -1.5708"/>
         <parent link="base_link"/>
-        <child link="akula_rig_link"/>
+        <child link="fin_link"/>
     </joint>
     <!-- ************************************************** -->

File: urdfs/tracer_links.xacro (robot description, xacro)
@@ -41,6 +41,6 @@
         <mesh filename="file://$(find tracer_ign_sim)/models/tracer/meshes/tracer_wheel.dae"/>
     </xacro:macro>
-    <xacro:macro name="akula_rig">
-        <mesh filename="file://$(find tracer_ign_sim)/models/tracer/meshes/tracer_sensor_rig.stl" scale="0.001 0.001 0.001"/>
+    <xacro:macro name="akula_fin_link">
+        <mesh filename="file://$(find tracer_ign_sim)/models/tracer/meshes/fin.stl" scale="0.001 0.001 0.001"/>
     </xacro:macro>
     <!-- Initial Link -->
@@ -282,11 +282,11 @@
         </collision>
     </link>
-    <link name="akula_rig_link">
-        <visual>
-            <geometry>
-                <xacro:akula_rig></xacro:akula_rig>
-            </geometry>
-            <material name="rig">
-                <color rgba="0.1 0.1 0.1 1"/>
+    <link name="fin_link">
+        <visual>
+            <geometry>
+                <xacro:akula_fin_link></xacro:akula_fin_link>
+            </geometry>
+            <material name="fin">
+                <color rgba="0.3 0.3 0.6 1"/>
             </material>
         </visual>
@@ -298,5 +298,5 @@
         <collision>
             <geometry>
-                <xacro:akula_rig></xacro:akula_rig>
+                <xacro:akula_fin_link></xacro:akula_fin_link>
             </geometry>
         </collision>
