Commit message: updated urdf with Velodyne VLP16 lidar sensor

File: urdfs/gazebo.xacro (robot description, xacro)
@@ -7,4 +7,6 @@
 -->
 <robot xmlns:xacro="http://www.ros.org/wiki/xacro">
+    <xacro:property name="M_PI" value="3.1415926535897931" />
+    <xacro:macro name="vlp16_scan_link" params="*origin parent:=base_link name:=velodyne topic:=/velodyne_points hz:=10 lasers:=16 samples:=1875 collision_range:=0.3 min_range:=0.2 max_range:=130.0 noise:=0.008 min_angle:=-${M_PI} max_angle:=${M_PI} gpu:=false">
     <gazebo reference="fl_wheel_link">
         <mu1>1</mu1>
@@ -31,3 +33,86 @@
         <slip2>0</slip2>
     </gazebo>
+    <!-- Gazebo requires the velodyne_gazebo_plugins package -->
+    <gazebo reference="${name}">
+      <xacro:if value="${gpu}">
+        <sensor type="gpu_ray" name="${name}-VLP16">
+          <pose>0 0 0 0 0 0</pose>
+          <visualize>false</visualize>
+          <update_rate>${hz}</update_rate>
+          <ray>
+            <scan>
+              <horizontal>
+                <samples>${samples}</samples>
+                <resolution>1</resolution>
+                <min_angle>${min_angle}</min_angle>
+                <max_angle>${max_angle}</max_angle>
+              </horizontal>
+              <vertical>
+                <samples>${lasers}</samples>
+                <resolution>1</resolution>
+                <min_angle>-${15.0*M_PI/180.0}</min_angle>
+                <max_angle> ${15.0*M_PI/180.0}</max_angle>
+              </vertical>
+            </scan>
+            <range>
+              <min>${collision_range}</min>
+              <max>${max_range+1}</max>
+              <resolution>0.001</resolution>
+            </range>
+            <noise>
+              <type>gaussian</type>
+              <mean>0.0</mean>
+              <stddev>0.0</stddev>
+            </noise>
+          </ray>
+          <plugin name="gazebo_ros_laser_controller" filename="libgazebo_ros_velodyne_gpu_laser.so">
+            <topicName>${topic}</topicName>
+            <frameName>${name}</frameName>
+            <min_range>${min_range}</min_range>
+            <max_range>${max_range}</max_range>
+            <gaussianNoise>${noise}</gaussianNoise>
+          </plugin>
+        </sensor>
+      </xacro:if>
+      <xacro:unless value="${gpu}">
+        <sensor type="ray" name="${name}-VLP16">
+          <pose>0 0 0 0 0 0</pose>
+          <visualize>false</visualize>
+          <update_rate>${hz}</update_rate>
+          <ray>
+            <scan>
+              <horizontal>
+                <samples>${samples}</samples>
+                <resolution>1</resolution>
+                <min_angle>${min_angle}</min_angle>
+                <max_angle>${max_angle}</max_angle>
+              </horizontal>
+              <vertical>
+                <samples>${lasers}</samples>
+                <resolution>1</resolution>
+                <min_angle>-${15.0*M_PI/180.0}</min_angle>
+                <max_angle> ${15.0*M_PI/180.0}</max_angle>
+              </vertical>
+            </scan>
+            <range>
+              <min>${collision_range}</min>
+              <max>${max_range+1}</max>
+              <resolution>0.001</resolution>
+            </range>
+            <noise>
+              <type>gaussian</type>
+              <mean>0.0</mean>
+              <stddev>0.0</stddev>
+            </noise>
+          </ray>
+          <plugin name="gazebo_ros_laser_controller" filename="libgazebo_ros_velodyne_laser.so">
+            <topicName>${topic}</topicName>
+            <frameName>${name}</frameName>
+            <min_range>${min_range}</min_range>
+            <max_range>${max_range}</max_range>
+            <gaussianNoise>${noise}</gaussianNoise>
+          </plugin>
+        </sensor>
+      </xacro:unless>
+    </gazebo>
 </robot>

File: urdfs/tracer_joints.xacro (robot description, xacro)
@@ -96,3 +96,14 @@
         <dynamics damping="0.2"/>
     </joint>
+    <!-- VLP16 lidar joint -->
+    <joint name="vlp16_fin_base_joint" type="fixed" >
+      <origin xyz="0 -0.15 0.83" rpy="0 0 3.14" />
+      <parent link="fin_link" />
+      <child link="vlp16_base_link"/>
+    </joint>
+    <joint name="vlp16_base_scan_joint" type="fixed" >
+      <origin xyz="0 0 0" rpy="0 0 0" />
+      <parent link="vlp16_base_link" />
+      <child link="vlp16_scan_link"/>
+    </joint>
 </robot>

File: urdfs/tracer_links.xacro (robot description, xacro)
@@ -44,4 +44,13 @@
         <mesh filename="file://$(find tracer_ign_sim)/models/tracer/meshes/fin.stl" scale="0.001 0.001 0.001"/>
     </xacro:macro>
+    <xacro:macro name="vlp16_base">
+        <mesh filename="file://$(find tracer_ign_sim)/models/tracer/meshes/VLP16/VLP16_base_1.stl"/>
+    </xacro:macro>
+    <xacro:macro name="vlp16_scan">
+        <mesh filename="file://$(find tracer_ign_sim)/models/tracer/meshes/VLP16/VLP16_scan.stl"/>
+    </xacro:macro>
+    <xacro:macro name="vlp16_top">
+        <mesh filename="file://$(find tracer_ign_sim)/models/tracer/meshes/VLP16/VLP16_base_2.stl"/>
+    </xacro:macro>
     <!-- Initial Link -->
     <link name="inertial_link">
@@ -288,5 +297,5 @@
             </geometry>
             <material name="fin">
-                <color rgba="0.3 0.3 0.6 1"/>
+                <color rgba="0.15 0.15 0.15 1"/>
             </material>
         </visual>
@@ -302,3 +311,54 @@
         </collision>
     </link>
+    <link name="vlp16_base_link">
+        <inertial>
+        <mass value="0.83"/>
+        <origin xyz="0 0 0.03585"/>
+        <inertia ixx="${(0.83 * (3.0*0.0516*0.0516 + 0.0717*0.0717)) / 12.0}" ixy="0" ixz="0"
+          iyy="${(0.83 * (3.0*0.0516*0.0516 + 0.0717*0.0717)) / 12.0}" iyz="0"
+          izz="${0.5 * 0.83 * (0.0516*0.0516)}"/>
+      </inertial>
+      <visual>
+        <geometry>
+            <xacro:vlp16_base></xacro:vlp16_base>
+        </geometry>
+        <material name="base1">
+                <color rgba="0.7 0.7 0.7 1"/>
+        </material>
+      </visual>
+      <visual>
+        <geometry>
+            <xacro:vlp16_top></xacro:vlp16_top>
+        </geometry>
+        <material name="base2">
+                <color rgba="0.7 0.7 0.7 1"/>
+        </material>
+      </visual>
+      <collision>
+        <origin rpy="0 0 0" xyz="0 0 0.03585"/>
+        <geometry>
+          <cylinder radius="0.0516" length="0.0717"/>
+        </geometry>
+      </collision>
+    </link>
+    <link name="vlp16_scan_link">
+        <visual>
+            <geometry>
+                <xacro:vlp16_scan></xacro:vlp16_scan>
+            </geometry>
+            <material name="scan">
+                <color rgba="0.1 0.1 0.3 1"/>
+            </material>
+        </visual>
+        <inertial>
+            <mass value="0.01" />
+            <origin xyz="0 0 0.03585" />
+            <inertia ixx="1e-7" ixy="0" ixz="0" iyy="1e-7" iyz="0" izz="1e-7"/>
+        </inertial>
+        <collision>
+            <geometry>
+                <xacro:vlp16_scan></xacro:vlp16_scan>
+            </geometry>
+        </collision>
+    </link>
 </robot>

Commit message: added lidar and imu

File: urdfs/gazebo.xacro (robot description, xacro)
@@ -6,7 +6,6 @@
     ========================================
 -->
-<robot xmlns:xacro="http://www.ros.org/wiki/xacro">
+<robot xmlns:xacro="http://www.ros.org/wiki/xacro" name="gazebo">
     <xacro:property name="M_PI" value="3.1415926535897931" />
-    <xacro:macro name="vlp16_scan_link" params="*origin parent:=base_link name:=velodyne topic:=/velodyne_points hz:=10 lasers:=16 samples:=1875 collision_range:=0.3 min_range:=0.2 max_range:=130.0 noise:=0.008 min_angle:=-${M_PI} max_angle:=${M_PI} gpu:=false">
     <gazebo reference="fl_wheel_link">
         <mu1>1</mu1>
@@ -33,86 +32,3 @@
         <slip2>0</slip2>
     </gazebo>
-    <!-- Gazebo requires the velodyne_gazebo_plugins package -->
-    <gazebo reference="${name}">
-      <xacro:if value="${gpu}">
-        <sensor type="gpu_ray" name="${name}-VLP16">
-          <pose>0 0 0 0 0 0</pose>
-          <visualize>false</visualize>
-          <update_rate>${hz}</update_rate>
-          <ray>
-            <scan>
-              <horizontal>
-                <samples>${samples}</samples>
-                <resolution>1</resolution>
-                <min_angle>${min_angle}</min_angle>
-                <max_angle>${max_angle}</max_angle>
-              </horizontal>
-              <vertical>
-                <samples>${lasers}</samples>
-                <resolution>1</resolution>
-                <min_angle>-${15.0*M_PI/180.0}</min_angle>
-                <max_angle> ${15.0*M_PI/180.0}</max_angle>
-              </vertical>
-            </scan>
-            <range>
-              <min>${collision_range}</min>
-              <max>${max_range+1}</max>
-              <resolution>0.001</resolution>
-            </range>
-            <noise>
-              <type>gaussian</type>
-              <mean>0.0</mean>
-              <stddev>0.0</stddev>
-            </noise>
-          </ray>
-          <plugin name="gazebo_ros_laser_controller" filename="libgazebo_ros_velodyne_gpu_laser.so">
-            <topicName>${topic}</topicName>
-            <frameName>${name}</frameName>
-            <min_range>${min_range}</min_range>
-            <max_range>${max_range}</max_range>
-            <gaussianNoise>${noise}</gaussianNoise>
-          </plugin>
-        </sensor>
-      </xacro:if>
-      <xacro:unless value="${gpu}">
-        <sensor type="ray" name="${name}-VLP16">
-          <pose>0 0 0 0 0 0</pose>
-          <visualize>false</visualize>
-          <update_rate>${hz}</update_rate>
-          <ray>
-            <scan>
-              <horizontal>
-                <samples>${samples}</samples>
-                <resolution>1</resolution>
-                <min_angle>${min_angle}</min_angle>
-                <max_angle>${max_angle}</max_angle>
-              </horizontal>
-              <vertical>
-                <samples>${lasers}</samples>
-                <resolution>1</resolution>
-                <min_angle>-${15.0*M_PI/180.0}</min_angle>
-                <max_angle> ${15.0*M_PI/180.0}</max_angle>
-              </vertical>
-            </scan>
-            <range>
-              <min>${collision_range}</min>
-              <max>${max_range+1}</max>
-              <resolution>0.001</resolution>
-            </range>
-            <noise>
-              <type>gaussian</type>
-              <mean>0.0</mean>
-              <stddev>0.0</stddev>
-            </noise>
-          </ray>
-          <plugin name="gazebo_ros_laser_controller" filename="libgazebo_ros_velodyne_laser.so">
-            <topicName>${topic}</topicName>
-            <frameName>${name}</frameName>
-            <min_range>${min_range}</min_range>
-            <max_range>${max_range}</max_range>
-            <gaussianNoise>${noise}</gaussianNoise>
-          </plugin>
-        </sensor>
-      </xacro:unless>
-    </gazebo>
 </robot>

File: urdfs/ros2_control.xacro (robot description, xacro)
@@ -61,7 +61,8 @@
     </ros2_control>
     <gazebo>
-        <!-- <plugin filename="libignition-gazebo-joint-state-publisher-system.so" name="ignition::gazebo::systems::JointStatePublisher"/> -->
-        <plugin filename="ign_ros2_control-system" name="ign_ros2_control::IgnitionROS2ControlPlugin">
-            <parameters>$(find tracer_ign_sim)/config/tracer_controller_velocity.yaml</parameters>
+        <plugin
+          filename="ign_ros2_control-system"
+          name="ign_ros2_control::IgnitionROS2ControlPlugin">
+          <parameters>$(find tracer_ign_sim)/config/tracer_controller_velocity.yaml</parameters>
         </plugin>
     </gazebo>

File: urdfs/tracer.urdf.xacro (robot description, xacro)
@@ -14,7 +14,9 @@
     <!-- ros2 control -->
     <xacro:include filename="$(find tracer_ign_sim)/urdfs/ros2_control.xacro"/>
-    <!-- <xacro:include filename="$(find tracer_ign_sim)/urdfs/gazebo.xacro"/> -->
-    <!-- <gazebo reference="L_wheel">
-        <mu1>0.2</mu1>
-    </gazebo> -->
+    <!-- gazebo -->
+    <xacro:include filename="$(find tracer_ign_sim)/urdfs/gazebo.xacro"/>
+    <!-- lidar -->
+    <xacro:include filename="$(find tracer_ign_sim)/urdfs/lidar.xacro"/>
+    <!-- imu -->
+    <xacro:include filename="$(find tracer_ign_sim)/urdfs/imu.xacro"/>
 </robot>

File: urdfs/tracer_joints.xacro (robot description, xacro)
@@ -97,4 +97,9 @@
     </joint>
     <!-- VLP16 lidar joint -->
+    <joint name="vlp16_base_scan_joint" type="fixed" >
+        <origin xyz="0 0 0" rpy="0 0 0" />
+        <parent link="vlp16_base_link" />
+        <child link="vlp16_scan"/>
+    </joint>
     <joint name="vlp16_fin_base_joint" type="fixed" >
       <origin xyz="0 -0.15 0.83" rpy="0 0 3.14" />
@@ -102,8 +107,3 @@
       <child link="vlp16_base_link"/>
     </joint>
-    <joint name="vlp16_base_scan_joint" type="fixed" >
-      <origin xyz="0 0 0" rpy="0 0 0" />
-      <parent link="vlp16_base_link" />
-      <child link="vlp16_scan_link"/>
-    </joint>
 </robot>

File: urdfs/tracer_links.xacro (robot description, xacro)
@@ -44,13 +44,4 @@
         <mesh filename="file://$(find tracer_ign_sim)/models/tracer/meshes/fin.stl" scale="0.001 0.001 0.001"/>
     </xacro:macro>
-    <xacro:macro name="vlp16_base">
-        <mesh filename="file://$(find tracer_ign_sim)/models/tracer/meshes/VLP16/VLP16_base_1.stl"/>
-    </xacro:macro>
-    <xacro:macro name="vlp16_scan">
-        <mesh filename="file://$(find tracer_ign_sim)/models/tracer/meshes/VLP16/VLP16_scan.stl"/>
-    </xacro:macro>
-    <xacro:macro name="vlp16_top">
-        <mesh filename="file://$(find tracer_ign_sim)/models/tracer/meshes/VLP16/VLP16_base_2.stl"/>
-    </xacro:macro>
     <!-- Initial Link -->
     <link name="inertial_link">
@@ -79,4 +70,10 @@
             </geometry>
         </collision>
+        <sensor name="imu_sensor" type="imu">
+            <always_on>1</always_on>
+            <update_rate>1</update_rate>
+            <visualize>true</visualize>
+            <topic>imu</topic>
+        </sensor>
     </link>
     <!-- ************************************************** -->
@@ -311,36 +308,46 @@
         </collision>
     </link>
+    <!-- Velodyne VLP16 -->
+    <xacro:macro name="vlp16_base">
+        <mesh filename="file://$(find tracer_ign_sim)/models/tracer/meshes/VLP16/VLP16_base_1.stl"/>
+    </xacro:macro>
+    <xacro:macro name="vlp16_scan">
+        <mesh filename="file://$(find tracer_ign_sim)/models/tracer/meshes/VLP16/VLP16_scan.stl"/>
+    </xacro:macro>
+    <xacro:macro name="vlp16_top">
+        <mesh filename="file://$(find tracer_ign_sim)/models/tracer/meshes/VLP16/VLP16_base_2.stl"/>
+    </xacro:macro>
     <link name="vlp16_base_link">
         <inertial>
-        <mass value="0.83"/>
-        <origin xyz="0 0 0.03585"/>
-        <inertia ixx="${(0.83 * (3.0*0.0516*0.0516 + 0.0717*0.0717)) / 12.0}" ixy="0" ixz="0"
-          iyy="${(0.83 * (3.0*0.0516*0.0516 + 0.0717*0.0717)) / 12.0}" iyz="0"
-          izz="${0.5 * 0.83 * (0.0516*0.0516)}"/>
-      </inertial>
-      <visual>
-        <geometry>
-            <xacro:vlp16_base></xacro:vlp16_base>
-        </geometry>
-        <material name="base1">
-                <color rgba="0.7 0.7 0.7 1"/>
-        </material>
-      </visual>
-      <visual>
-        <geometry>
-            <xacro:vlp16_top></xacro:vlp16_top>
-        </geometry>
-        <material name="base2">
-                <color rgba="0.7 0.7 0.7 1"/>
-        </material>
-      </visual>
-      <collision>
-        <origin rpy="0 0 0" xyz="0 0 0.03585"/>
-        <geometry>
-          <cylinder radius="0.0516" length="0.0717"/>
-        </geometry>
-      </collision>
-    </link>
-    <link name="vlp16_scan_link">
+            <mass value="0.83"/>
+            <origin xyz="0 0 0.03585"/>
+            <inertia ixx="${(0.83 * (3.0*0.0516*0.0516 + 0.0717*0.0717)) / 12.0}" ixy="0" ixz="0"
+            iyy="${(0.83 * (3.0*0.0516*0.0516 + 0.0717*0.0717)) / 12.0}" iyz="0"
+            izz="${0.5 * 0.83 * (0.0516*0.0516)}"/>
+        </inertial>
+        <visual>
+            <geometry>
+                <xacro:vlp16_base></xacro:vlp16_base>
+            </geometry>
+            <material name="base1">
+                    <color rgba="0.7 0.7 0.7 1"/>
+            </material>
+        </visual>
+        <visual>
+            <geometry>
+                <xacro:vlp16_top></xacro:vlp16_top>
+            </geometry>
+            <material name="base2">
+                    <color rgba="0.7 0.7 0.7 1"/>
+            </material>
+        </visual>
+        <collision>
+            <origin rpy="0 0 0" xyz="0 0 0.03585"/>
+            <geometry>
+            <cylinder radius="0.0516" length="0.0717"/>
+            </geometry>
+        </collision>
+    </link>
+    <link name="vlp16_scan">
         <visual>
             <geometry>
