Commit message: finalizaed ign lidar sim with ros_ign_bridge

File: urdfs/lidar.xacro (robot description, xacro)
@@ -3,5 +3,5 @@
     <xacro:property name="M_PI" value="3.1415926535897931" />
     <xacro:property name="name" value="velodyne" />
-    <xacro:property name="topic" value="vlp16" />
+    <xacro:property name="topic" value="lidar" />
     <xacro:property name="organize_cloud" value="false" />
     <xacro:property name="hz" value="10" />
@@ -18,5 +18,5 @@
         <xacro:if value="${gpu}">
             <sensor name="lidar_ray" type="gpu_ray">
-                <pose relative_to='vlp16_scan'>0 0 0 0 0 0</pose>
+                <pose>0 0 0 0 0 0</pose>
                 <topic>${topic}</topic>
                 <update_rate>${hz}</update_rate>
@@ -58,5 +58,5 @@
         <xacro:unless value="${gpu}">
             <sensor name="lidar_ray" type="lidar">
-                <pose relative_to='vlp16_scan'>0 0 0 0 0 0</pose>
+                <pose>0 0 0 0 0 0</pose>
                 <topic>${topic}</topic>
                 <update_rate>${hz}</update_rate>

File: urdfs/tracer.urdf.xacro (robot description, xacro)
@@ -19,4 +19,4 @@
     <xacro:include filename="$(find tracer_ign_sim)/urdfs/lidar.xacro"/>
     <!-- imu -->
-    <xacro:include filename="$(find tracer_ign_sim)/urdfs/imu.xacro"/>
+    <!-- <xacro:include filename="$(find tracer_ign_sim)/urdfs/imu.xacro"/> -->
 </robot>
