Commit message: Updated the pkg name and added rviz to launch file

File: urdfs/akula.urdf.xacro (robot description, xacro)
@@ -6,16 +6,16 @@
    ========================================
 -->
-<robot xmlns:xacro="http://www.ros.org/wiki/xacro"  name="tracer">
+<robot xmlns:xacro="http://www.ros.org/wiki/xacro"  name="Akula">
     <origin xyz="0 0 0.3" rpy="0 0 0"/>
     <!-- links -->
-    <xacro:include filename="$(find tracer_ign_sim)/urdfs/tracer_links.xacro" />
+    <xacro:include filename="$(find akula_ign_sim)/urdfs/akula_links.xacro" />
     <!-- joints -->
-    <xacro:include filename="$(find tracer_ign_sim)/urdfs/tracer_joints.xacro" />
+    <xacro:include filename="$(find akula_ign_sim)/urdfs/akula_joints.xacro" />
     <!-- ros2 control -->
-    <xacro:include filename="$(find tracer_ign_sim)/urdfs/ros2_control.xacro"/>
+    <xacro:include filename="$(find akula_ign_sim)/urdfs/ros2_control.xacro"/>
     <!-- gazebo -->
-    <xacro:include filename="$(find tracer_ign_sim)/urdfs/gazebo.xacro"/>
+    <xacro:include filename="$(find akula_ign_sim)/urdfs/gazebo.xacro"/>
     <!-- lidar -->
-    <xacro:include filename="$(find tracer_ign_sim)/urdfs/lidar.xacro"/>
+    <xacro:include filename="$(find akula_ign_sim)/urdfs/velodyne_VLP16.xacro"/>
     <!-- imu -->
     <!-- <xacro:include filename="$(find tracer_ign_sim)/urdfs/imu.xacro"/> -->

File: urdfs/akula_joints.xacro (robot description, xacro)
@@ -6,5 +6,5 @@
     ========================================
 -->
-<robot>
+<robot xmlns:xacro="http://www.ros.org/wiki/xacro" name="Akula joints">
     <joint name="base_joint" type="fixed">
         <origin xyz="0 0 0" rpy="0 0 0"/>

File: urdfs/akula_links.xacro (robot description, xacro)
@@ -6,5 +6,5 @@
     ========================================
 -->
-<robot xmlns:xacro="http://www.ros.org/wiki/xacro">
+<robot xmlns:xacro="http://www.ros.org/wiki/xacro" name="Akula links">
     <!-- load meshes -->
     <xacro:macro name="base_link">

File: urdfs/gazebo.xacro (robot description, xacro)
@@ -7,5 +7,4 @@
 -->
 <robot xmlns:xacro="http://www.ros.org/wiki/xacro" name="gazebo">
-    <xacro:property name="M_PI" value="3.1415926535897931" />
     <gazebo reference="fl_wheel_link">
         <mu1>1</mu1>

File: urdfs/imu.xacro (robot description, xacro)
@@ -1,3 +1,9 @@
 <?xml version="1.0"?>
+<!--
+    ========================================
+      * Author: nipun.dhananjaya@gmail.com
+      * Created: 04.2023
+    ========================================
+-->
 <robot xmlns:xacro="http://www.ros.org/wiki/xacro" name="imu">
     <gazebo reference="base_link">

File: urdfs/ros2_control.xacro (robot description, xacro)
@@ -6,5 +6,5 @@
     ========================================
 -->
-<robot xmlns:xacro="http://www.ros.org/wiki/xacro">
+<robot xmlns:xacro="http://www.ros.org/wiki/xacro" name="ros2_control">
     <ros2_control name="IgnitionSystem" type="system">
         <hardware>

File: urdfs/velodyne_VLP16.xacro (robot description, xacro)
@@ -1,13 +1,19 @@
 <?xml version="1.0"?>
+<!--
+    ========================================
+      * Author: nipun.dhananjaya@gmail.com
+      * Created: 04.2023
+    ========================================
+-->
 <robot xmlns:xacro="http://www.ros.org/wiki/xacro" name="vlp16">
     <xacro:property name="M_PI" value="3.1415926535897931" />
     <xacro:property name="name" value="velodyne" />
-    <xacro:property name="topic" value="lidar" />
+    <xacro:property name="topic" value="/velodyne" />
     <xacro:property name="organize_cloud" value="false" />
     <xacro:property name="hz" value="10" />
     <xacro:property name="lasers" value="16" />
     <xacro:property name="samples" value="1875" />
-    <xacro:property name="collision_range" value="0.3" />
-    <xacro:property name="min_range" value="0.9" />
+    <xacro:property name="collision_range" value="0.7" />
+    <xacro:property name="min_range" value="0.3" />
     <xacro:property name="max_range" value="130.0 " />
     <xacro:property name="noise" value="0.008" />
@@ -17,5 +23,5 @@
     <gazebo reference="vlp16_scan">
         <xacro:if value="${gpu}">
-            <sensor name="lidar_ray" type="gpu_ray">
+            <sensor name="velodyne-VLP16" type="gpu_ray">
                 <pose>0 0 0 0 0 0</pose>
                 <topic>${topic}</topic>
@@ -57,5 +63,5 @@
         </xacro:if>
         <xacro:unless value="${gpu}">
-            <sensor name="lidar_ray" type="lidar">
+            <sensor name="velodyne-VLP16" type="ray">
                 <pose>0 0 0 0 0 0</pose>
                 <topic>${topic}</topic>

Commit message: updated

File: urdfs/akula.urdf.xacro (robot description, xacro)
@@ -6,5 +6,5 @@
    ========================================
 -->
-<robot xmlns:xacro="http://www.ros.org/wiki/xacro"  name="Akula">
+<robot xmlns:xacro="http://www.ros.org/wiki/xacro"  name="akula">
     <origin xyz="0 0 0.3" rpy="0 0 0"/>
     <!-- links -->

File: urdfs/akula_links.xacro (robot description, xacro)
@@ -9,38 +9,38 @@
     <!-- load meshes -->
     <xacro:macro name="base_link">
-        <mesh filename="file://$(find tracer_ign_sim)/models/tracer/meshes/tracer_base_link_no_wheel.dae"/>
+        <mesh filename="file://$(find akula_ign_sim)/models/tracer/meshes/tracer_base_link_no_wheel.dae"/>
     </xacro:macro>
     <xacro:macro name="fl_castor_link">
-        <mesh filename="file://$(find tracer_ign_sim)/models/tracer/meshes/castor_joint.dae"/>
+        <mesh filename="file://$(find akula_ign_sim)/models/tracer/meshes/castor_joint.dae"/>
     </xacro:macro>
     <xacro:macro name="fr_castor_link">
-        <mesh filename="file://$(find tracer_ign_sim)/models/tracer/meshes/castor_joint.dae"/>
+        <mesh filename="file://$(find akula_ign_sim)/models/tracer/meshes/castor_joint.dae"/>
     </xacro:macro>
     <xacro:macro name="rl_castor_link">
-        <mesh filename="file://$(find tracer_ign_sim)/models/tracer/meshes/castor_joint.dae"/>
+        <mesh filename="file://$(find akula_ign_sim)/models/tracer/meshes/castor_joint.dae"/>
     </xacro:macro>
     <xacro:macro name="rr_castor_link">
-        <mesh filename="file://$(find tracer_ign_sim)/models/tracer/meshes/castor_joint.dae"/>
+        <mesh filename="file://$(find akula_ign_sim)/models/tracer/meshes/castor_joint.dae"/>
     </xacro:macro>
     <xacro:macro name="fl_wheel_link">
-        <mesh filename="file://$(find tracer_ign_sim)/models/tracer/meshes/castor.dae"/>
+        <mesh filename="file://$(find akula_ign_sim)/models/tracer/meshes/castor.dae"/>
     </xacro:macro>
     <xacro:macro name="fr_wheel_link">
-        <mesh filename="file://$(find tracer_ign_sim)/models/tracer/meshes/castor.dae"/>
+        <mesh filename="file://$(find akula_ign_sim)/models/tracer/meshes/castor.dae"/>
     </xacro:macro>
     <xacro:macro name="rl_wheel_link">
-        <mesh filename="file://$(find tracer_ign_sim)/models/tracer/meshes/castor.dae"/>
+        <mesh filename="file://$(find akula_ign_sim)/models/tracer/meshes/castor.dae"/>
     </xacro:macro>
     <xacro:macro name="rr_wheel_link">
-        <mesh filename="file://$(find tracer_ign_sim)/models/tracer/meshes/castor.dae"/>
+        <mesh filename="file://$(find akula_ign_sim)/models/tracer/meshes/castor.dae"/>
     </xacro:macro>
     <xacro:macro name="L_wheel_link">
-        <mesh filename="file://$(find tracer_ign_sim)/models/tracer/meshes/tracer_wheel.dae"/>
+        <mesh filename="file://$(find akula_ign_sim)/models/tracer/meshes/tracer_wheel.dae"/>
     </xacro:macro>
     <xacro:macro name="R_wheel_link">
-        <mesh filename="file://$(find tracer_ign_sim)/models/tracer/meshes/tracer_wheel.dae"/>
+        <mesh filename="file://$(find akula_ign_sim)/models/tracer/meshes/tracer_wheel.dae"/>
     </xacro:macro>
     <xacro:macro name="akula_fin_link">
-        <mesh filename="file://$(find tracer_ign_sim)/models/tracer/meshes/fin.stl" scale="0.001 0.001 0.001"/>
+        <mesh filename="file://$(find akula_ign_sim)/models/tracer/meshes/fin.stl" scale="0.001 0.001 0.001"/>
     </xacro:macro>
     <!-- Initial Link -->
@@ -310,11 +310,11 @@
     <!-- Velodyne VLP16 -->
     <xacro:macro name="vlp16_base">
-        <mesh filename="file://$(find tracer_ign_sim)/models/tracer/meshes/VLP16/VLP16_base_1.stl"/>
+        <mesh filename="file://$(find akula_ign_sim)/models/tracer/meshes/VLP16/VLP16_base_1.stl"/>
     </xacro:macro>
     <xacro:macro name="vlp16_scan">
-        <mesh filename="file://$(find tracer_ign_sim)/models/tracer/meshes/VLP16/VLP16_scan.stl"/>
+        <mesh filename="file://$(find akula_ign_sim)/models/tracer/meshes/VLP16/VLP16_scan.stl"/>
     </xacro:macro>
     <xacro:macro name="vlp16_top">
-        <mesh filename="file://$(find tracer_ign_sim)/models/tracer/meshes/VLP16/VLP16_base_2.stl"/>
+        <mesh filename="file://$(find akula_ign_sim)/models/tracer/meshes/VLP16/VLP16_base_2.stl"/>
     </xacro:macro>
     <link name="vlp16_base_link">

File: urdfs/ros2_control.xacro (robot description, xacro)
@@ -64,5 +64,5 @@
           filename="ign_ros2_control-system"
           name="ign_ros2_control::IgnitionROS2ControlPlugin">
-          <parameters>$(find tracer_ign_sim)/config/tracer_controller_velocity.yaml</parameters>
+          <parameters>$(find akula_ign_sim)/config/tracer_controller_velocity.yaml</parameters>
         </plugin>
     </gazebo>
