Commit message: made seperate pkgs for description and ignition

File: akula_description/urdf/akula.urdf.xacro (robot description, xacro)
@@ -9,13 +9,13 @@
     <origin xyz="0 0 0.3" rpy="0 0 0"/>
     <!-- links -->
-    <xacro:include filename="$(find akula_ign_sim)/urdfs/akula_links.xacro" />
+    <xacro:include filename="$(find akula_description)/urdf/akula_links.xacro" />
     <!-- joints -->
-    <xacro:include filename="$(find akula_ign_sim)/urdfs/akula_joints.xacro" />
+    <xacro:include filename="$(find akula_description)/urdf/akula_joints.xacro" />
     <!-- ros2 control -->
-    <xacro:include filename="$(find akula_ign_sim)/urdfs/ros2_control.xacro"/>
+    <xacro:include filename="$(find akula_description)/urdf/ros2_control.xacro"/>
     <!-- gazebo -->
-    <xacro:include filename="$(find akula_ign_sim)/urdfs/gazebo.xacro"/>
+    <xacro:include filename="$(find akula_description)/urdf/gazebo.xacro"/>
     <!-- lidar -->
-    <xacro:include filename="$(find akula_ign_sim)/urdfs/velodyne_VLP16.xacro"/>
+    <xacro:include filename="$(find akula_description)/urdf/velodyne_VLP16.xacro"/>
     <!-- imu -->
     <!-- <xacro:include filename="$(find tracer_ign_sim)/urdfs/imu.xacro"/> -->

File: akula_description/urdf/akula_joints.xacro (robot description, xacro)
@@ -16,4 +16,9 @@
         <parent link="base_link"/>
         <child link="fin_link"/>
+    </joint>
+    <joint name="base_footprint_joint" type="fixed">
+        <parent link="base_link"/>
+        <child link="base_footprint"/>
+        <origin xyz="0 0 0" pry="0 0 0"/>
     </joint>
     <!-- ************************************************** -->
@@ -96,14 +101,3 @@
         <dynamics damping="0.2"/>
     </joint>
-    <!-- VLP16 lidar joint -->
-    <joint name="vlp16_base_scan_joint" type="fixed" >
-        <origin xyz="0 0 0" rpy="0 0 0" />
-        <parent link="vlp16_base_link" />
-        <child link="vlp16_scan"/>
-    </joint>
-    <joint name="vlp16_fin_base_joint" type="fixed" >
-      <origin xyz="0 -0.15 0.83" rpy="0 0 3.14" />
-      <parent link="fin_link" />
-      <child link="vlp16_base_link"/>
-    </joint>
 </robot>

File: akula_description/urdf/akula_links.xacro (robot description, xacro)
@@ -9,38 +9,38 @@
     <!-- load meshes -->
     <xacro:macro name="base_link">
-        <mesh filename="file://$(find akula_ign_sim)/models/tracer/meshes/tracer_base_link_no_wheel.dae"/>
+        <mesh filename="file://$(find akula_description)/meshes/tracer_base_link_no_wheel.dae"/>
     </xacro:macro>
     <xacro:macro name="fl_castor_link">
-        <mesh filename="file://$(find akula_ign_sim)/models/tracer/meshes/castor_joint.dae"/>
+        <mesh filename="file://$(find akula_description)/meshes/castor_joint.dae"/>
     </xacro:macro>
     <xacro:macro name="fr_castor_link">
-        <mesh filename="file://$(find akula_ign_sim)/models/tracer/meshes/castor_joint.dae"/>
+        <mesh filename="file://$(find akula_description)/meshes/castor_joint.dae"/>
     </xacro:macro>
     <xacro:macro name="rl_castor_link">
-        <mesh filename="file://$(find akula_ign_sim)/models/tracer/meshes/castor_joint.dae"/>
+        <mesh filename="file://$(find akula_description)/meshes/castor_joint.dae"/>
     </xacro:macro>
     <xacro:macro name="rr_castor_link">
-        <mesh filename="file://$(find akula_ign_sim)/models/tracer/meshes/castor_joint.dae"/>
+        <mesh filename="file://$(find akula_description)/meshes/castor_joint.dae"/>
     </xacro:macro>
     <xacro:macro name="fl_wheel_link">
-        <mesh filename="file://$(find akula_ign_sim)/models/tracer/meshes/castor.dae"/>
+        <mesh filename="file://$(find akula_description)/meshes/castor.dae"/>
     </xacro:macro>
     <xacro:macro name="fr_wheel_link">
-        <mesh filename="file://$(find akula_ign_sim)/models/tracer/meshes/castor.dae"/>
+        <mesh filename="file://$(find akula_description)/meshes/castor.dae"/>
     </xacro:macro>
     <xacro:macro name="rl_wheel_link">
-        <mesh filename="file://$(find akula_ign_sim)/models/tracer/meshes/castor.dae"/>
+        <mesh filename="file://$(find akula_description)/meshes/castor.dae"/>
     </xacro:macro>
     <xacro:macro name="rr_wheel_link">
-        <mesh filename="file://$(find akula_ign_sim)/models/tracer/meshes/castor.dae"/>
+        <mesh filename="file://$(find akula_description)/meshes/castor.dae"/>
     </xacro:macro>
     <xacro:macro name="L_wheel_link">
-        <mesh filename="file://$(find akula_ign_sim)/models/tracer/meshes/tracer_wheel.dae"/>
+        <mesh filename="file://$(find akula_description)/meshes/tracer_wheel.dae"/>
     </xacro:macro>
     <xacro:macro name="R_wheel_link">
-        <mesh filename="file://$(find akula_ign_sim)/models/tracer/meshes/tracer_wheel.dae"/>
+        <mesh filename="file://$(find akula_description)/meshes/tracer_wheel.dae"/>
     </xacro:macro>
     <xacro:macro name="akula_fin_link">
-        <mesh filename="file://$(find akula_ign_sim)/models/tracer/meshes/fin.stl" scale="0.001 0.001 0.001"/>
+        <mesh filename="file://$(find akula_description)/meshes/fin.stl" scale="0.001 0.001 0.001"/>
     </xacro:macro>
     <!-- Initial Link -->
@@ -77,4 +77,5 @@
         </sensor>
     </link>
+    <link name="base_footprint"></link>
     <!-- ************************************************** -->
     <!-- FL castor joint link -->
@@ -308,64 +309,3 @@
         </collision>
     </link>
-    <!-- Velodyne VLP16 -->
-    <xacro:macro name="vlp16_base">
-        <mesh filename="file://$(find akula_ign_sim)/models/tracer/meshes/VLP16/VLP16_base_1.stl"/>
-    </xacro:macro>
-    <xacro:macro name="vlp16_scan">
-        <mesh filename="file://$(find akula_ign_sim)/models/tracer/meshes/VLP16/VLP16_scan.stl"/>
-    </xacro:macro>
-    <xacro:macro name="vlp16_top">
-        <mesh filename="file://$(find akula_ign_sim)/models/tracer/meshes/VLP16/VLP16_base_2.stl"/>
-    </xacro:macro>
-    <link name="vlp16_base_link">
-        <inertial>
-            <mass value="0.83"/>
-            <origin xyz="0 0 0.03585"/>
-            <inertia ixx="${(0.83 * (3.0*0.0516*0.0516 + 0.0717*0.0717)) / 12.0}" ixy="0" ixz="0"
-            iyy="${(0.83 * (3.0*0.0516*0.0516 + 0.0717*0.0717)) / 12.0}" iyz="0"
-            izz="${0.5 * 0.83 * (0.0516*0.0516)}"/>
-        </inertial>
-        <visual>
-            <geometry>
-                <xacro:vlp16_base></xacro:vlp16_base>
-            </geometry>
-            <material name="base1">
-                    <color rgba="0.7 0.7 0.7 1"/>
-            </material>
-        </visual>
-        <visual>
-            <geometry>
-                <xacro:vlp16_top></xacro:vlp16_top>
-            </geometry>
-            <material name="base2">
-                    <color rgba="0.7 0.7 0.7 1"/>
-            </material>
-        </visual>
-        <collision>
-            <origin rpy="0 0 0" xyz="0 0 0.03585"/>
-            <geometry>
-            <cylinder radius="0.0516" length="0.0717"/>
-            </geometry>
-        </collision>
-    </link>
-    <link name="vlp16_scan">
-        <visual>
-            <geometry>
-                <xacro:vlp16_scan></xacro:vlp16_scan>
-            </geometry>
-            <material name="scan">
-                <color rgba="0.1 0.1 0.3 1"/>
-            </material>
-        </visual>
-        <inertial>
-            <mass value="0.01" />
-            <origin xyz="0 0 0.03585" />
-            <inertia ixx="1e-7" ixy="0" ixz="0" iyy="1e-7" iyz="0" izz="1e-7"/>
-        </inertial>
-        <collision>
-            <geometry>
-                <xacro:vlp16_scan></xacro:vlp16_scan>
-            </geometry>
-        </collision>
-    </link>
 </robot>

File: akula_description/urdf/velodyne_VLP16.xacro (robot description, xacro)
@@ -21,4 +21,78 @@
     <xacro:property name="max_angle" value="${M_PI}" />
     <xacro:property name="gpu" value="true"/>
+    <!-- Velodyne VLP16 -->
+    <xacro:macro name="vlp16_base">
+        <mesh filename="file://$(find akula_description)/meshes/VLP16/VLP16_base_1.stl"/>
+    </xacro:macro>
+    <xacro:macro name="vlp16_scan">
+        <mesh filename="file://$(find akula_description)/meshes/VLP16/VLP16_scan.stl"/>
+    </xacro:macro>
+    <xacro:macro name="vlp16_top">
+        <mesh filename="file://$(find akula_description)/meshes/VLP16/VLP16_base_2.stl"/>
+    </xacro:macro>
+    <!-- LINKS -->
+    <link name="vlp16_base_link">
+        <inertial>
+            <mass value="0.83"/>
+            <origin xyz="0 0 0.03585"/>
+            <inertia ixx="${(0.83 * (3.0*0.0516*0.0516 + 0.0717*0.0717)) / 12.0}" ixy="0" ixz="0"
+            iyy="${(0.83 * (3.0*0.0516*0.0516 + 0.0717*0.0717)) / 12.0}" iyz="0"
+            izz="${0.5 * 0.83 * (0.0516*0.0516)}"/>
+        </inertial>
+        <visual>
+            <geometry>
+                <xacro:vlp16_base></xacro:vlp16_base>
+            </geometry>
+            <material name="base1">
+                    <color rgba="0.7 0.7 0.7 1"/>
+            </material>
+        </visual>
+        <visual>
+            <geometry>
+                <xacro:vlp16_top></xacro:vlp16_top>
+            </geometry>
+            <material name="base2">
+                    <color rgba="0.7 0.7 0.7 1"/>
+            </material>
+        </visual>
+        <collision>
+            <origin rpy="0 0 0" xyz="0 0 0.03585"/>
+            <geometry>
+            <cylinder radius="0.0516" length="0.0717"/>
+            </geometry>
+        </collision>
+    </link>
+    <link name="vlp16_scan">
+        <visual>
+            <geometry>
+                <xacro:vlp16_scan></xacro:vlp16_scan>
+            </geometry>
+            <material name="scan">
+                <color rgba="0.1 0.1 0.3 1"/>
+            </material>
+        </visual>
+        <inertial>
+            <mass value="0.01" />
+            <origin xyz="0 0 0.03585" />
+            <inertia ixx="1e-7" ixy="0" ixz="0" iyy="1e-7" iyz="0" izz="1e-7"/>
+        </inertial>
+        <collision>
+            <geometry>
+                <xacro:vlp16_scan></xacro:vlp16_scan>
+            </geometry>
+        </collision>
+    </link>
+    <!-- VLP16 lidar joint -->
+    <joint name="vlp16_fin_base_joint" type="fixed" >
+      <origin xyz="0 -0.15 0.83" rpy="0 0 3.14" />
+      <parent link="fin_link" />
+      <child link="vlp16_base_link"/>
+    </joint>
+    <joint name="vlp16_base_scan_joint" type="fixed" >
+        <origin xyz="0 0 0" rpy="0 0 0" />
+        <parent link="vlp16_base_link" />
+        <child link="vlp16_scan"/>
+    </joint>
+    <!-- GAZEBO PLUGIN -->
     <gazebo reference="vlp16_scan">
         <xacro:if value="${gpu}">

Commit message: added imu sensor, camera

File: akula_description/urdf/akula.urdf.xacro (robot description, xacro)
@@ -19,4 +19,6 @@
     <xacro:include filename="$(find akula_description)/urdf/velodyne_VLP16.xacro"/>
     <!-- imu -->
-    <!-- <xacro:include filename="$(find tracer_ign_sim)/urdfs/imu.xacro"/> -->
+    <xacro:include filename="$(find akula_description)/urdf/imu.xacro"/>
+    <!-- camera -->
+    <xacro:include filename="$(find akula_description)/urdf/camera.xacro"/>
 </robot>

File: akula_description/urdf/akula_links.xacro (robot description, xacro)
@@ -295,5 +295,5 @@
             </geometry>
             <material name="fin">
-                <color rgba="0.15 0.15 0.15 1"/>
+                <color rgba="0.058 0.058 0.058 1"/>
             </material>
         </visual>

File: akula_description/urdf/velodyne_VLP16.xacro (robot description, xacro)
@@ -85,5 +85,5 @@
     <!-- VLP16 lidar joint -->
     <joint name="vlp16_fin_base_joint" type="fixed" >
-      <origin xyz="0 -0.15 0.83" rpy="0 0 3.14" />
+      <origin xyz="0 -0.15 0.855" rpy="0 0 3.14" />
       <parent link="fin_link" />
       <child link="vlp16_base_link"/>
@@ -97,5 +97,5 @@
     <gazebo reference="vlp16_scan">
         <xacro:if value="${gpu}">
-            <sensor name="velodyne-VLP16" type="gpu_ray">
+            <sensor name="VLP16" type="gpu_ray">
                 <pose>0 0 0 0 0 0</pose>
                 <topic>${topic}</topic>
@@ -137,5 +137,5 @@
         </xacro:if>
         <xacro:unless value="${gpu}">
-            <sensor name="velodyne-VLP16" type="ray">
+            <sensor name="VLP16" type="ray">
                 <pose>0 0 0 0 0 0</pose>
                 <topic>${topic}</topic>
