Commit message: camera is fixed

File: akula_description/urdf/camera.xacro (robot description, xacro)
@@ -40,12 +40,13 @@
         <parent link="camera_link"/>
         <child link="camera_optical_link"/>
-        <origin xyz="0 0 0" rpy="${-pi/2} 0 ${-pi/2}"/>
+        <origin xyz="0 0 0" rpy="0 0 ${-pi/2}"/>
     </joint>
     <link name="camera_optical_link"></link>
-    <gazebo reference="camera_link">
+    <gazebo reference="camera_optical_link">
         <sensor name="camera" type="camera">
             <pose> 0 0 0 0 0 0 </pose>
             <visualize>true</visualize>
             <update_rate>10</update_rate>
+            <topic>camera</topic>
             <camera>
                 <horizontal_fov>1.089</horizontal_fov>
