Commit message: urdf update

File: akula_description/urdf/velodyne_VLP16.xacro (robot description, xacro)
@@ -8,6 +8,6 @@
 <robot xmlns:xacro="http://www.ros.org/wiki/xacro" name="vlp16">
     <xacro:property name="M_PI" value="3.1415926535897931" />
-    <xacro:property name="name" value="velodyne" />
-    <xacro:property name="topic" value="/velodyne" />
+    <xacro:property name="name" value="velodyne_sim" />
+    <xacro:property name="topic" value="/vlp16_sim_scan" />
     <xacro:property name="organize_cloud" value="false" />
     <xacro:property name="hz" value="10" />
@@ -79,5 +79,5 @@
         <collision>
             <geometry>
-                <xacro:vlp16_scan></xacro:vlp16_scan>
+                <sphere radius="0"/>
             </geometry>
         </collision>
@@ -101,4 +101,5 @@
                 <topic>${topic}</topic>
                 <update_rate>${hz}</update_rate>
+                <frame_name>${name}</frame_name>
                 <ray>
                     <scan>
@@ -173,4 +174,5 @@
                     name="ignition::gazebo::systems::Sensors">
                     <render_engine>ogre</render_engine>
+                    <frame_name>${name}</frame_name>
                 </plugin>
             </sensor>
