Commit message: configured akula_description pkg to work with slam_toolbox

File: akula_description/urdf/akula_joints.xacro (robot description, xacro)
@@ -7,4 +7,9 @@
 -->
 <robot xmlns:xacro="http://www.ros.org/wiki/xacro" name="Akula joints">
+    <joint name="base_footprint_joint" type="fixed">
+        <parent link="base_footprint"/>
+        <child link="base_link"/>
+        <origin xyz="0 0 0" pry="0 0 0"/>
+    </joint>
     <joint name="base_joint" type="fixed">
         <origin xyz="0 0 0" rpy="0 0 0"/>
@@ -16,9 +21,4 @@
         <parent link="base_link"/>
         <child link="fin_link"/>
-    </joint>
-    <joint name="base_footprint_joint" type="fixed">
-        <parent link="base_link"/>
-        <child link="base_footprint"/>
-        <origin xyz="0 0 0" pry="0 0 0"/>
     </joint>
     <!-- ************************************************** -->

File: akula_description/urdf/akula_links.xacro (robot description, xacro)
@@ -44,4 +44,5 @@
         <mesh filename="file://$(find akula_description)/meshes/fin.stl" scale="0.001 0.001 0.001"/>
     </xacro:macro>
+    <link name="base_footprint"></link>
     <!-- Initial Link -->
     <link name="inertial_link">
@@ -77,5 +78,4 @@
         </sensor>
     </link>
-    <link name="base_footprint"></link>
     <!-- ************************************************** -->
     <!-- FL castor joint link -->
